File: _autosave-Credit Card PCB V1.kicad_sch (KiCad schematic)
At the start: 37 parts, among them SW1 SW_Push, SW2 RotaryEncoder, U1 ATmega32U4-A, Y1 16MHz

Commit message: Update
Parts:
- added J1: USB_C_Receptacle_USB2.0, symbol Connector:USB_C_Receptacle_USB2.0
- added U2: ATmega32U2-A, Package_QFP:TQFP-32_7x7mm_P0.8mm, symbol MCU_Microchip_ATmega:ATmega32U2-A
Connections:
- new net: J1.A1 (GND), J1.A12 (GND), J1.B1 (GND), J1.B12 (GND)
- new net: J1.A4 (VBUS), J1.A9 (VBUS), J1.B4 (VBUS), J1.B9 (VBUS)
Other:
- moved on the sheet: C2, C3, C4, C5, SW2
