File: _autosave-Credit Card PCB V1.kicad_sch (KiCad schematic)
At the start: 53 parts, among them J1 USB_C_Receptacle_USB2.0, SW0 SW_Push, SW1 RotaryEncoder, U1 USBLC6-2SC6, U2 ATmega32U2-A, Y1 16MHz

Commit message: Large Update
Parts:
- H0, H1, H2, H3: footprint (none) -> MountingHole:MountingHole_2.2mm_M2_Pad_Via
Changed lines of the file:
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@@
       (effects (font (size 1.27 1.27)) (justify left))
     )
-    (property "Footprint" "" (at 191.77 102.87 0)
+    (property "Footprint" "MountingHole:MountingHole_2.2mm_M2_Pad_Via" (at 191.77 102.87 0)
       (effects (font (size 1.27 1.27)) hide)
     )
@@
       (effects (font (size 1.27 1.27)) (justify left))
     )
-    (property "Footprint" "" (at 147.32 102.87 0)
+    (property "Footprint" "MountingHole:MountingHole_2.2mm_M2_Pad_Via" (at 147.32 102.87 0)
       (effects (font (size 1.27 1.27)) hide)
     )
@@
       (effects (font (size 1.27 1.27)) (justify left))
     )
-    (property "Footprint" "" (at 213.36 102.87 0)
+    (property "Footprint" "MountingHole:MountingHole_2.2mm_M2_Pad_Via" (at 213.36 102.87 0)
       (effects (font (size 1.27 1.27)) hide)
     )
@@
       (effects (font (size 1.27 1.27)) (justify left))
     )
-    (property "Footprint" "" (at 170.18 102.87 0)
-      (effects (font (size 1.27 1.27)) hide)
-    )
+    (property "Footprint" "MountingHole:MountingHole_2.2mm_M2_Pad_Via" (at 170.18 102.87 0)
+      (effects (font (size 1.27 1.27)) hide)
+    )
