File: Credit Card PCB V1.kicad_sch (KiCad schematic)
At the start: 53 parts, among them J1 USB_C_Receptacle_USB2.0, SW0 SW_Push, SW1 RotaryEncoder, U1 USBLC6-2SC6, U2 ATmega32U2-A, Y1 16MHz

Commit message: Another Chunky Update
Parts:
- F1: footprint Fuse:Fuse_0603_1608Metric -> Fuse:Fuse_1206_3216Metric
- H0, H1, H2, H3: footprint (none) -> MountingHole:MountingHole_2.2mm_M2_Pad_Via
- R5, R6: value R_Small -> 5.1k
- SW0: footprint Button_Switch_SMD:SW_SPST_EVQP7C -> Button_Switch_SMD:SW_SPST_SKQG_WithStem
Changed lines of the file:
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@@
       (effects (font (size 1.27 1.27)) (justify left))
     )
-    (property "Footprint" "" (at 191.77 102.87 0)
+    (property "Footprint" "MountingHole:MountingHole_2.2mm_M2_Pad_Via" (at 191.77 102.87 0)
       (effects (font (size 1.27 1.27)) hide)
     )
@@
       (effects (font (size 1.27 1.27)) (justify left))
     )
-    (property "Footprint" "" (at 147.32 102.87 0)
+    (property "Footprint" "MountingHole:MountingHole_2.2mm_M2_Pad_Via" (at 147.32 102.87 0)
       (effects (font (size 1.27 1.27)) hide)
     )
@@
       (effects (font (size 1.27 1.27)))
     )
-    (property "Footprint" "Button_Switch_SMD:SW_SPST_EVQP7C" (at 40.64 81.28 0)
+    (property "Footprint" "Button_Switch_SMD:SW_SPST_SKQG_WithStem" (at 40.64 81.28 0)
       (effects (font (size 1.27 1.27)) hide)
     )
@@
       (effects (font (size 1.27 1.27)))
     )
-    (property "Footprint" "Fuse:Fuse_0603_1608Metric" (at 180.34 133.35 0)
+    (property "Footprint" "Fuse:Fuse_1206_3216Metric" (at 180.34 133.35 0)
       (effects (font (size 1.27 1.27)) (justify left) hide)
     )
@@
       (effects (font (size 1.27 1.27)))
     )
-    (property "Value" "R_Small" (at 30.48 49.53 90)
+    (property "Value" "5.1k" (at 30.48 49.53 90)
       (effects (font (size 1.27 1.27)))
     )
@@
       (effects (font (size 1.27 1.27)) (justify left))
     )
-    (property "Footprint" "" (at 213.36 102.87 0)
+    (property "Footprint" "MountingHole:MountingHole_2.2mm_M2_Pad_Via" (at 213.36 102.87 0)
       (effects (font (size 1.27 1.27)) hide)
     )
@@
       (effects (font (size 1.27 1.27)) (justify left))
     )
-    (property "Footprint" "" (at 170.18 102.87 0)
+    (property "Footprint" "MountingHole:MountingHole_2.2mm_M2_Pad_Via" (at 170.18 102.87 0)
       (effects (font (size 1.27 1.27)) hide)
     )
@@
       (effects (font (size 1.27 1.27)))
     )
-    (property "Value" "R_Small" (at 30.48 57.15 90)
-      (effects (font (size 1.27 1.27)))
-    )
+    (property "Value" "5.1k" (at 30.48 57.15 90)
+      (effects (font (size 1.27 1.27)))
+    )

Commit message: Just a couple small things
Parts:
- J1: footprint Connector_USB:USB_C_Receptacle_GCT_USB4105-xx-A_16P_TopMnt_Horizontal -> keyswitches.pretty-master:GCT_USB4110-GF-A_REVB
Changed lines of the file:
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@@
       (effects (font (size 1.27 1.27)))
     )
-    (property "Footprint" "Connector_USB:USB_C_Receptacle_GCT_USB4105-xx-A_16P_TopMnt_Horizontal" (at 46.99 44.45 0)
+    (property "Footprint" "keyswitches.pretty-master:GCT_USB4110-GF-A_REVB" (at 46.99 44.45 0)
       (effects (font (size 1.27 1.27)) hide)
     )
